Commit message: add kinect sensor in urdf

File: urdf/my_robot_tutorial.urdf (robot description, URDF)
Before this commit: robot my_robot, 7 links, 6 joints
Links:
- added link camera_link_optical
- added link depth_image_link, mass 0.035; collision box size=0.008 0.130 0.022; visual box size=0.008 0.130 0.022
Joints:
- added joint camera_optical_joint: type fixed, parent depth_image_link, child camera_link_optical, origin xyz=0 0 0 rpy=-1.570796326 0 -1.570796326
- added joint image_joint: type fixed, parent base_link, child depth_image_link, origin xyz=0.70 0 0.175 rpy=0 0 0
